File: schematics/bike_computer/bike_computer.kicad_pcb (KiCad board)
At the start: 2 copper layers, 0 parts

Commit message: bike computer layout v0
Parts:
- added 3.3V: 3V3, FahrradTech:TestPoint_Keystone_5000-5004_Miniature, F.Cu at (105.5, 51.4)
- added BT1: Battery_Cell, FahrradTech:BatteryHolder_18650, B.Cu at (89.3, 47.0)
- added C1: 0.1uF, Capacitor_THT:C_Rect_L4.6mm_W2.0mm_P2.50mm_MKS02_FKP02, F.Cu at (169.1, 62.7)
- added C2: 470pF, Capacitor_THT:C_Rect_L4.6mm_W2.0mm_P2.50mm_MKS02_FKP02, F.Cu at (118.3, 60.5)
- added C3: 10uF, Capacitor_THT:CP_Radial_D5.0mm_P2.00mm, B.Cu at (111.6, 51.4)
- added C4: 0.1uF, Capacitor_THT:C_Rect_L4.6mm_W2.0mm_P2.50mm_MKS02_FKP02, F.Cu at (154.2, 106.9)
- added C5: 0.1uF, Capacitor_THT:C_Rect_L4.6mm_W2.0mm_P2.50mm_MKS02_FKP02, F.Cu at (81.4, 64.4)
- added C6: 0.1uF, Capacitor_THT:C_Rect_L4.6mm_W2.0mm_P2.50mm_MKS02_FKP02, F.Cu at (122.2, 116.4)
- added C7: 10uF, Capacitor_THT:CP_Radial_D5.0mm_P2.00mm, B.Cu at (124.7, 50.2)
- added G***: LOGO, FahrradTech:resisty_0.5x0.65inch, B.Cu at (171.5, 53.4)
- added GND: GND, FahrradTech:TestPoint_Keystone_5000-5004_Miniature, B.Cu at (103.5, 113.3)
- added R1: 121k, Resistor_THT:R_Axial_DIN0207_L6.3mm_D2.5mm_P10.16mm_Horizontal, F.Cu at (88.5, 74.8)
- added R2: 40.2k, Resistor_THT:R_Axial_DIN0207_L6.3mm_D2.5mm_P10.16mm_Horizontal, F.Cu at (98.6, 66.5)
- added REF**: 2mm, MountingHole:MountingHole_2mm, F.Cu at (178.9, 121.3)
- added REF**: 2mm, MountingHole:MountingHole_2mm, F.Cu at (72.9, 121.3)
- added REF**: 2mm, MountingHole:MountingHole_2mm, F.Cu at (178.9, 48.3)
- added REF**: 2mm, MountingHole:MountingHole_2mm, F.Cu at (72.9, 48.3)
- added SW1: GW12LxH, FahrradTech:SW_Lever_1P2T_NKK_GW12LxH, B.Cu at (132.2, 53.2)
- added U2: BME280, FahrradTech:BME280_module, B.Cu at (166.4, 68.1)
- added U3: TC1263, FahrradTech:TO-220-5_P3.4x3.8mm_StaggerOdd_Lead7.13mm_TabDown, F.Cu at (122.4, 60.4)
- added U4: TFT LCD ST7796, FahrradTech:Display_420x380, F.Cu at (73.8, 70.6)
- added U5: TP4056 module, FahrradTech:TP4056_module, F.Cu at (83.1, 122.1)
- added U6: RYS352A, FahrradTech:RYS352A, B.Cu at (140.7, 94.0)
- added U7: ESP-WROOM-32-DevKitV1, FahrradTech:ESP-WROOM-32_DevKitV1, B.Cu at (109.5, 113.9)
- added VBATT: VBATT, FahrradTech:TestPoint_Keystone_5000-5004_Miniature, B.Cu at (103.3, 95.1)
Routing:
- net GND: track 0.00 -> 296.1 mm
- net +3.3V: track 0.00 -> 241.0 mm
- net Net-(U4-SDI(MOSI)): track 0.00 -> 161.7 mm
- net Net-(U4-SDO(MISO)): track 0.00 -> 153.9 mm
- net Net-(U4-SCK): track 0.00 -> 133.8 mm
- net Net-(U5-OUT+): track 0.00 -> 112.2 mm
- net Net-(U4-RESET_N): track 0.00 -> 82.0 mm
- net Net-(U4-DC/RS): track 0.00 -> 80.0 mm
- net CS: track 0.00 -> 79.7 mm
- net Net-(U4-T_IRQ_N): track 0.00 -> 74.8 mm
- net Net-(U4-LED): track 0.00 -> 72.8 mm
- net SD_CS: track 0.00 -> 71.3 mm
- net Net-(U2-SCK): track 0.00 -> 69.0 mm
- net Net-(U4-T_CS): track 0.00 -> 64.1 mm
- net Net-(U2-SDI): track 0.00 -> 58.3 mm
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Other:
- board outline added: 112 x 79 mm
- board text added: "FahrradTech Bike Computer v0"
