File: schematics/rear_lights_unit_control_box/rear_lights_unit_control_box.kicad_sch (KiCad schematic)
At the start: 11 parts, among them J1 Conn_01x04_Socket, SW1 SW_SPDT, SW2 SW_SPDT

Commit message: updated both sets of light unit board files to include the newly-added 3D models
Parts:
- TP1, TP2, TP3, TP4: footprint TestPoint:TestPoint_Keystone_5000-5004_Miniature -> FahrradTech:TestPoint_Keystone_5000-5004_Miniature
Other:
- title: FarrhadTech Rear Lights Unit Control Box -> FahrradTech Rear Lights Unit Control Box
Changed lines of the file:
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@@
 	(paper "A4")
 	(title_block
-		(title "FarrhadTech Rear Lights Unit Control Box")
+		(title "FahrradTech Rear Lights Unit Control Box")
 		(date "2025-03-31")
 	)
@@
 			)
 		)
-		(property "Footprint" "TestPoint:TestPoint_Keystone_5000-5004_Miniature"
+		(property "Footprint" "FahrradTech:TestPoint_Keystone_5000-5004_Miniature"
 			(at 69.342 40.64 0)
 			(effects
@@
 			)
 		)
-		(property "Footprint" "TestPoint:TestPoint_Keystone_5000-5004_Miniature"
+		(property "Footprint" "FahrradTech:TestPoint_Keystone_5000-5004_Miniature"
 			(at 83.566 43.18 0)
 			(effects
@@
 			)
 		)
-		(property "Footprint" "TestPoint:TestPoint_Keystone_5000-5004_Miniature"
+		(property "Footprint" "FahrradTech:TestPoint_Keystone_5000-5004_Miniature"
 			(at 111.76 48.26 0)
 			(effects
@@
 			)
 		)
-		(property "Footprint" "TestPoint:TestPoint_Keystone_5000-5004_Miniature"
+		(property "Footprint" "FahrradTech:TestPoint_Keystone_5000-5004_Miniature"
 			(at 97.536 45.72 0)
 			(effects
